Commit message: Added PointCloud2 definition for roboception camera

File: rc_visard_driver/urdf/rc_visard65.gazebo.xacro (robot description, xacro)
@@ -2,8 +2,8 @@
 <robot xmlns:xacro="http://ros.org/wiki/xacro">
 	<xacro:macro name="rc_visard65_stereo_gazebo" params="link_name frame_name camera_name camera_type camera_rate">
-		<xacro:unless value="${camera_type == 'color'}">
+		<xacro:if value="${camera_type == 'monochrome'}">
 			<xacro:property name="image_topic_suffix" value="" />
 			<xacro:property name="image_format" value="L8" />
-		</xacro:unless>
+		</xacro:if>
 		<xacro:if value="${camera_type == 'color'}">
 			<xacro:property name="image_topic_suffix" value="_color" />
@@ -60,6 +60,6 @@
 					<alwaysOn>true</alwaysOn>
 					<updateRate>0.0</updateRate>
-					<cameraName>${camera_name}_stereo</cameraName>
-					<imageTopicName>image_rect</imageTopicName>
+					<cameraName>${camera_name}/stereo/</cameraName>
+					<imageTopicName>image_rect${image_topic_suffix}</imageTopicName>
 					<cameraInfoTopicName>camera_info</cameraInfoTopicName>
 					<frameName>left_camera_optical_frame</frameName>
@@ -76,8 +76,8 @@
 	</xacro:macro>
 	<xacro:macro name="rc_visard65_depth_gazebo" params="link_name frame_name camera_name camera_type camera_rate">
-		<xacro:unless value="${camera_type == 'color'}">
+		<xacro:if value="${camera_type == 'monochrome'}">
 			<xacro:property name="image_topic_suffix" value="" />
 			<xacro:property name="image_format" value="L8" />
-		</xacro:unless>
+		</xacro:if>
 		<xacro:if value="${camera_type == 'color'}">
 			<xacro:property name="image_topic_suffix" value="_color" />
@@ -119,10 +119,10 @@
 					<alwaysOn>true</alwaysOn>
 					<updateRate>${image_rate}</updateRate>
-					<cameraName>${camera_name}_depth</cameraName>
-					<!--imageTopicName>/${camera_name}/depth/image_raw</imageTopicName-->
+					<cameraName>${camera_name}</cameraName>
+					<imageTopicName>/${camera_name}/rgb/image_raw</imageTopicName>
 					<depthImageTopicName>/${camera_name}/stereo/depth</depthImageTopicName>
 					<pointCloudTopicName>/${camera_name}/stereo/points2</pointCloudTopicName>
 					<frameName>${frame_name}</frameName>
-					<pointCloudCutoff>0.5</pointCloudCutoff>
+					<pointCloudCutoff>0.3</pointCloudCutoff>
 					<distortionK1>0.00000001</distortionK1>
 					<distortionK2>0.00000001</distortionK2>

File: rc_visard_driver/urdf/rc_visard65.urdf.xacro (robot description, xacro)
@@ -5,10 +5,10 @@
     <!-- rc_visard65 mount assembly -->
     <xacro:macro name="rc_visard65" params="name parent *origin camera_type camera_rate">
-        <joint name="${name}_rc_visard65_joint" type="fixed">
+        <joint name="${name}_joint" type="fixed">
             <xacro:insert_block name="origin" />
             <parent link="${parent}"/>
-            <child link="${name}_rc_visard65_link"/>
+            <child link="${name}_link"/>
         </joint>
-        <link name="${name}_rc_visard65_link">
+        <link name="${name}_link">
             <inertial>
                 <mass value="0.1"/>
@@ -35,10 +35,10 @@
         </link>
         <!-- rc_visard65 stereo sensor physical attachment -->
-        <joint name="${name}_rc_visard65_stereo_joint" type="fixed">
-            <origin xyz="-0.023 0.0325 0.0375" rpy="0 0 1.5708"/>
-            <parent link="${name}_rc_visard65_link"/>
-            <child link="${name}_rc_visard65_stereo_link"/>
+        <joint name="${name}_stereo_joint" type="fixed">
+            <origin xyz="-0.0325 0.0325 0.0375" rpy="0 0 1.5708"/>
+            <parent link="${name}_link"/>
+            <child link="${name}_stereo_link"/>
         </joint>
-        <link name="${name}_rc_visard65_stereo_link">
+        <link name="${name}_stereo_link">
             <inertial>
                 <mass value="0.1" />
@@ -61,21 +61,27 @@
             </collision>
         </link>
-        <!-- kinect2 ir sensor frame -->
-        <joint name="${name}_rc_visard65_stereo_optical_frame_joint" type="fixed">
-            <origin xyz="0 0 0" rpy="0 0 0" />
-            <parent link="${name}_rc_visard65_stereo_link"/>
-            <child link="${name}_rc_visard65_stereo_optical_frame"/>
+        <!-- rc_visard65 stereo sensor frame -->
+        <joint name="${name}_stereo_optical_frame_joint" type="fixed">
+            <origin xyz="0 0 0" rpy="${-PI/2} 0 ${-PI/2}" />
+            <parent link="${name}_stereo_link"/>
+            <child link="${name}_stereo_optical_frame"/>
         </joint>
-        <link name="${name}_rc_visard65_stereo_optical_frame"/>
+        <link name="${name}_stereo_optical_frame"/>
+        <joint name="${name}_stereo_right_frame_joint" type="fixed">
+            <origin xyz="0.065 0 0" rpy="0 0 0" />
+            <parent link="${name}_stereo_optical_frame"/>
+            <child link="${name}_stereo_right_optical_frame"/>
+        </joint>
+        <link name="${name}_stereo_right_optical_frame"/>
         <!-- gazebo extensions -->
-        <xacro:rc_visard65_stereo_gazebo link_name="${name}_rc_visard65_stereo_link" frame_name="${name}_rc_visard65_stereo_optical_frame" camera_name="rc_visard65"
+        <xacro:rc_visard65_stereo_gazebo link_name="${name}_stereo_link" frame_name="${name}_stereo_optical_frame" camera_name="${name}"
             camera_type="${camera_type}" camera_rate="${camera_rate}" />
-        <!-- kinect2 rgb sensor physical attachment
-        <joint name="${name}_kinect2_rgb_joint" type="fixed">
-            <origin xyz="0 -0.05175 0" rpy="0 0 0"/>
-            <parent link="${name}_kinect2_ir_link"/>
-            <child link="${name}_kinect2_rgb_link"/>
+        <!-- rc_visard65 point cloud sensor physical attachment -->
+        <joint name="${name}_pc_joint" type="fixed">
+            <origin xyz="0 0 0" rpy="0 0 0"/>
+            <parent link="${name}_stereo_link"/>
+            <child link="${name}_pc_link"/>
         </joint>
-        <link name="${name}_kinect2_rgb_link" >
+        <link name="${name}_pc_link" >
             <inertial>
                 <mass value="0.1" />
@@ -86,6 +92,5 @@
             </inertial>
             <visual>
-                <origin xyz="${cal_kinect_x}            ${cal_kinect_y}                 ${cal_kinect_z}"
-                    rpy="${-M_PI/2+cal_kinect_roll} ${0.0+cal_kinect_pitch}         ${-M_PI/2+cal_kinect_yaw}" />
+                <origin xyz="0 0 0" rpy="0 0 0" />
                 <geometry>
                     <sphere radius="0.0005"/>
@@ -98,15 +103,14 @@
                 </geometry>
             </collision>
-        </link>-->
-        <!-- kinect2 rgb sensor frame
-        <joint name="${name}_kinect2_rgb_optical_frame_joint" type="fixed">
-            <origin xyz="${cal_kinect_x}            ${cal_kinect_y}                 ${cal_kinect_z}"
-                rpy="${-M_PI/2+cal_kinect_roll} ${0.0+cal_kinect_pitch}         ${-M_PI/2+cal_kinect_yaw}" />
-                <parent link="${name}_kinect2_rgb_link"/>
-                <child link="${name}_kinect2_rgb_optical_frame"/>
+        </link>
+        <!-- rc_visard65 point cloud sensor frame -->
+        <joint name="${name}_pc_optical_frame_joint" type="fixed">
+            <origin xyz="0 0 0" rpy="${-PI/2} 0 ${-PI/2}" />
+                <parent link="${name}_pc_link"/>
+                <child link="${name}_pc_optical_frame"/>
         </joint>
-        <link name="${name}_kinect2_rgb_optical_frame"/>-->
-        <!-- gazebo extensions
-        <xacro:kinect2_rgb_gazebo_v0 link_name="${name}_kinect2_rgb_link" frame_name="${name}_kinect2_rgb_optical_frame" camera_name="head_mount_kinect2" />-->
+        <link name="${name}_pc_optical_frame"/>
+        <!-- gazebo extensions -->
+        <xacro:rc_visard65_depth_gazebo link_name="${name}_pc_link" frame_name="${name}_pc_optical_frame" camera_name="${name}" camera_type="${camera_type}" camera_rate="${camera_rate}" />
     </xacro:macro>
 </robot>

Commit message: Updated README to reflect added Gazebo simulation

File: rc_visard_driver/urdf/rc_visard65.gazebo.xacro (robot description, xacro)
@@ -3,9 +3,7 @@
 	<xacro:macro name="rc_visard65_stereo_gazebo" params="link_name frame_name camera_name camera_type camera_rate">
 		<xacro:if value="${camera_type == 'monochrome'}">
-			<xacro:property name="image_topic_suffix" value="" />
 			<xacro:property name="image_format" value="L8" />
 		</xacro:if>
 		<xacro:if value="${camera_type == 'color'}">
-			<xacro:property name="image_topic_suffix" value="_color" />
 			<xacro:property name="image_format" value="R8G8B8" />
 		</xacro:if>
@@ -61,5 +59,5 @@
 					<updateRate>0.0</updateRate>
 					<cameraName>${camera_name}/stereo/</cameraName>
-					<imageTopicName>image_rect${image_topic_suffix}</imageTopicName>
+					<imageTopicName>image_rect</imageTopicName>
 					<cameraInfoTopicName>camera_info</cameraInfoTopicName>
 					<frameName>left_camera_optical_frame</frameName>
