Commit message: Added reference frame for roboception images in rviz

File: rc_visard_driver/urdf/rc_visard65.urdf.xacro (robot description, xacro)
@@ -111,4 +111,11 @@
         </joint>
         <link name="${name}_pc_optical_frame"/>
+        <!-- create virtual frame for showing live camera images -->
+        <joint name="${name}_virtual_camera_joint" type="fixed">
+            <origin xyz="0 0 0" rpy="0 0 0" />
+                <parent link="${name}_pc_optical_frame"/>
+                <child link="${name}_camera"/>
+        </joint>
+        <link name="${name}_camera"/>
         <!-- gazebo extensions -->
         <xacro:rc_visard65_depth_gazebo link_name="${name}_pc_link" frame_name="${name}_pc_optical_frame" camera_name="${name}" camera_type="${camera_type}" camera_rate="${camera_rate}" />

Commit message: Fix for submodule definitions

File: rc_visard_driver/urdf/rc_visard65.urdf.xacro (robot description, xacro)
@@ -19,5 +19,5 @@
             </inertial>
             <visual>
-                <origin xyz="-0.023 0.0325 0.0375" rpy="-1.5708 0 0"/>
+                <origin xyz="-0.023 0.0325 0.0375" rpy="-${PI/2} 0 0"/>
                 <geometry>
                     <mesh filename="package://rc_visard_driver/meshes/rc_visard65.stl" scale="0.001 0.001 0.001" />
@@ -36,5 +36,5 @@
         <!-- rc_visard65 stereo sensor physical attachment -->
         <joint name="${name}_stereo_joint" type="fixed">
-            <origin xyz="-0.0325 0.0325 0.0375" rpy="0 0 1.5708"/>
+            <origin xyz="-0.0325 0.0325 0.0375" rpy="0 0 ${PI/2}"/>
             <parent link="${name}_link"/>
             <child link="${name}_stereo_link"/>

Commit message: Added collision hull for roboception

File: rc_visard_driver/urdf/rc_visard65.urdf.xacro (robot description, xacro)
@@ -1,4 +1,4 @@
 <?xml version="1.0"?>
-<robot xmlns:xacro="http://ros.org/wiki/xacro">
+<robot xmlns:xacro="http://www.ros.org/wiki/xacro">
     <xacro:include filename="$(find rc_visard_driver)/urdf/rc_visard65.gazebo.xacro" />
     <xacro:include filename="$(find rc_visard_driver)/urdf/rc_visard65_properties.urdf.xacro" />
@@ -23,12 +23,12 @@
                     <mesh filename="package://rc_visard_driver/meshes/rc_visard65.stl" scale="0.001 0.001 0.001" />
                 </geometry>
-                <material name="gray">
-                    <color rgba="0.5 0.5 0.5 1"/>
+                <material name="darkgray">
+                    <color rgba="0.3 0.3 0.3 1"/>
                 </material>
             </visual>
             <collision>
-                <origin xyz="0.0325 0 0.0315" rpy="0 0 0"/>
+                <origin xyz="0 -0.01 0.04" rpy="0 0 0"/>
                 <geometry>
-                    <sphere radius="0.0005"/>
+                    <box size="0.14 0.15 0.08"/>
                 </geometry>
             </collision>

Commit message: FIXED Points2Publisher now utilizes the correct timebase [ros::Time::now()] ADDED Parameter for simulation of the camera images in .xacro

File: rc_visard_driver/urdf/rc_visard65.urdf.xacro (robot description, xacro)
@@ -4,5 +4,5 @@
     <xacro:include filename="$(find rc_visard_driver)/urdf/rc_visard65_properties.urdf.xacro" />
     <!-- rc_visard65 mount assembly -->
-    <xacro:macro name="rc_visard65" params="name parent *origin camera_type camera_rate">
+    <xacro:macro name="rc_visard65" params="name parent *origin camera_type camera_rate simulated">
         <joint name="${name}_joint" type="fixed">
             <xacro:insert_block name="origin" />
@@ -75,6 +75,8 @@
         <link name="${name}_stereo_right_optical_frame"/>
         <!-- gazebo extensions -->
-        <xacro:rc_visard65_stereo_gazebo link_name="${name}_stereo_link" frame_name="${name}_stereo_optical_frame" camera_name="${name}"
-            camera_type="${camera_type}" camera_rate="${camera_rate}" />
+        <xacro:if value="${simulated}">
+            <xacro:rc_visard65_stereo_gazebo link_name="${name}_stereo_link" frame_name="${name}_stereo_optical_frame" camera_name="${name}"
+                camera_type="${camera_type}" camera_rate="${camera_rate}" />
+        </xacro:if>
         <!-- rc_visard65 point cloud sensor physical attachment -->
         <joint name="${name}_pc_joint" type="fixed">
@@ -119,5 +121,8 @@
         <link name="${name}_camera"/>
         <!-- gazebo extensions -->
-        <xacro:rc_visard65_depth_gazebo link_name="${name}_pc_link" frame_name="${name}_pc_optical_frame" camera_name="${name}" camera_type="${camera_type}" camera_rate="${camera_rate}" />
+        <xacro:if value="${simulated}">
+            <xacro:rc_visard65_depth_gazebo link_name="${name}_pc_link" frame_name="${name}_pc_optical_frame" camera_name="${name}" camera_type="${camera_type}"
+                camera_rate="${camera_rate}" />
+        </xacro:if>
     </xacro:macro>
 </robot>
